Commit message: update imu mpu9250

File: sensors/imu_mpu9250/imu_mpu9250.xacro (robot description, xacro)
@@ -2,5 +2,5 @@
 <robot name="imu_mpu9250"
     xmlns:xacro="http://ros.org/wiki/xacro">
-    <xacro:macro name="imu_mpu9250" params="prefix parent *origin">
+    <xacro:macro name="imu_mpu9250" params="prefix parent *origin prefix_topic">
         <joint name="${prefix}_fixed" type="fixed">
             <insert_block name="origin"/>
@@ -27,25 +27,21 @@
         <gazebo reference="${prefix}_frame">
             <gravity>true</gravity>
-            <plugin filename="libhector_gazebo_ros_imu.so" name="gazebo_ros_imu">
-                <bodyName>${prefix}_frame</bodyName>
-                <updateRate>50</updateRate>
-                <serviceName>imu_service</serviceName>
-                <topicName>imu</topicName>
-                <gaussianNoise>0</gaussianNoise>
-                <xyzOffset>0 0 0</xyzOffset>
-                <rpyOffset>0 0 0</rpyOffset>
-            </plugin>
+            <sensor name="${prefix}_sensor" type="imu">
+                <pose>0 0 0 0 0 0</pose>
+                <update_rate>10</update_rate>
+                <visualize>true</visualize>
+                <always_on>true</always_on>
+                <topic>__default_topic__</topic>
+                <plugin  name="${prefix}_gazebo_plugin" filename="libgazebo_ros_imu_sensor.so">
+                    <topicName>${prefix_topic}/imu</topicName>
+                    <bodyName>base_link</bodyName>
+                    <updateRateHZ>10.0</updateRateHZ>
+                    <gaussianNoise>0.0</gaussianNoise>
+                    <xyzOffset>0 0 0</xyzOffset>
+                    <rpyOffset>0 0 0</rpyOffset>
+                    <frameName>${prefix}_frame</frameName>
+                </plugin>
+            </sensor>
         </gazebo>
-        <!-- <gazebo reference="${prefix}_frame">
-            <gravity>true</gravity>
-            <plugin name="${prefix}_controller" filename="libgazebo_ros_imu.so">
-                <alwaysOn>true</alwaysOn>
-                <topicName>imu/data</topicName>
-                <serviceName>imu/service</serviceName>
-                <bodyName>${prefix}_frame</bodyName>
-                <updateRateHZ>50.0</updateRateHZ>
-                <gaussianNoise>0.005</gaussianNoise>
-            </plugin>
-        </gazebo> -->
     </xacro:macro>
 </robot>

File: sensors/ydlidar/ydlidar_g4.xacro (robot description, xacro)
@@ -64,10 +64,10 @@
                         <type>gaussian</type>
                         <mean>0.0</mean>
-                        <stddev>0.0025</stddev>
+                        <stddev>0.01</stddev>
                     </noise>
                 </ray>
                 <plugin name="${prefix}_gazebo_plugin" filename="libgazebo_ros_laser.so">
                     <topicName>${prefix_topic}/scan</topicName>
-                    <frameName>/${prefix}_frame</frameName>
+                    <frameName>${prefix}_frame</frameName>
                 </plugin>
             </sensor>

Commit message: update

File: sensors/imu_mpu9250/imu_mpu9250.xacro (robot description, xacro)
@@ -30,7 +30,4 @@
                 <pose>0 0 0 0 0 0</pose>
                 <update_rate>10</update_rate>
-                <visualize>true</visualize>
-                <always_on>true</always_on>
-                <topic>__default_topic__</topic>
                 <plugin  name="${prefix}_gazebo_plugin" filename="libgazebo_ros_imu_sensor.so">
                     <topicName>${prefix_topic}/imu</topicName>

File: sensors/intel_realsense_d435/intel_realsense_d435.xacro (robot description, xacro)
@@ -21,32 +21,32 @@
     <xacro:property name="d435_cam_depth_py" value="0.0175"/>
     <xacro:property name="d435_cam_depth_pz" value="${d435_cam_height/2}"/>
-    <link name="base_link"/>
-    <!-- camera body, with origin at bottom screw mount -->
-    <joint name="camera_joint" type="fixed">
-        <!-- <xacro:insert_block name="origin" /> -->
-        <parent link="base_link"/>
-        <child link="camera_link" />
-    </joint>
-    <link name="camera_link">
-        <visual>
-            <origin xyz="${d435_cam_mount_from_center_offset} 0.0 ${d435_cam_height/2}" rpy="${M_PI/2} 0 ${M_PI/2}"/>
-            <geometry>
-                <mesh filename="package://anman_sensors/sensors/intel_realsense_d435/meshes/d435.dae" />
-            </geometry>
-            <material name="aluminum"/>
-        </visual>
-        <collision>
-            <origin xyz="0.0 0.0 ${d435_cam_height/2}" rpy="0 0 0"/>
-            <geometry>
-                <box size="${d435_cam_depth} ${d435_cam_width} ${d435_cam_height}"/>
-            </geometry>
-        </collision>
-        <inertial>
-            <!-- The following are not reliable values, and should not be used for modeling -->
-            <mass value="0.564" />
-            <origin xyz="0 0 0" />
-            <inertia ixx="0.003881243" ixy="0.0" ixz="0.0" iyy="0.000498940" iyz="0.0" izz="0.003879257" />
-        </inertial>
-    </link>
+    <xacro:macro name="intel_realsense_d435" params="prefix parent *origin prefix_topic">
+        <joint name="${prefix}_camera_fixed" type="fixed">
+            <insert_block name="origin"/>
+            <parent link="${parent}"/>
+            <child link="${prefix}_camera_frame"/>
+        </joint>
+        <link name="${prefix}_camera_frame">
+            <visual>
+                <origin xyz="${d435_cam_mount_from_center_offset} 0.0 ${d435_cam_height/2}" rpy="${M_PI/2} 0 ${M_PI/2}"/>
+                <geometry>
+                    <mesh filename="package://anman_sensors/sensors/intel_realsense_d435/meshes/d435.dae" />
+                </geometry>
+                <material name="aluminum"/>
+            </visual>
+            <collision>
+                <origin xyz="0.0 0.0 ${d435_cam_height/2}" rpy="0 0 0"/>
+                <geometry>
+                    <box size="${d435_cam_depth} ${d435_cam_width} ${d435_cam_height}"/>
+                </geometry>
+            </collision>
+            <inertial>
+                <!-- The following are not reliable values, and should not be used for modeling -->
+                <mass value="0.564" />
+                <origin xyz="0 0 0" />
+                <inertia ixx="0.003881243" ixy="0.0" ixz="0.0" iyy="0.000498940" iyz="0.0" izz="0.003879257" />
+            </inertial>
+        </link>
+    </xacro:macro>
     <!-- camera depth joints and links -->
     <joint name="camera_depth_joint" type="fixed">

Commit message: change imu frame to link

File: sensors/imu_mpu9250/imu_mpu9250.xacro (robot description, xacro)
@@ -6,7 +6,7 @@
             <insert_block name="origin"/>
             <parent link="${parent}"/>
-            <child link="${prefix}_frame"/>
+            <child link="${prefix}_link"/>
         </joint>
-        <link name="${prefix}_frame">
+        <link name="${prefix}_link">
             <visual>
                 <origin xyz="0 0 0" rpy="0 0 0"/>
@@ -25,5 +25,5 @@
             <box_inertia m="0.01" x="0.02" y="0.02" z="0.02"/>
         </link>
-        <gazebo reference="${prefix}_frame">
+        <gazebo reference="${prefix}_link">
             <gravity>true</gravity>
             <sensor name="${prefix}_sensor" type="imu">
@@ -37,5 +37,5 @@
                     <xyzOffset>0 0 0</xyzOffset>
                     <rpyOffset>0 0 0</rpyOffset>
-                    <frameName>${prefix}_frame</frameName>
+                    <frameName>${prefix}_link</frameName>
                 </plugin>
             </sensor>
