Commit message: update

File: materials.xacro (robot description, xacro)
@@ -1,4 +1,4 @@
 <?xml version="1.0"?>
-<robot>
+<robot xmlns:xacro="http://ros.org/wiki/xacro">
     <material name="black">
         <color rgba="0.0 0.0 0.0 1.0"/>
@@ -28,3 +28,12 @@
         <color rgba="0.5 0.5 0.5 1.0"/>
     </material>
+    <xacro:macro name="cylinder_inertia" params="m r h">
+        <inertia ixx="${m*(3*r*r+h*h)/12}" ixy = "0" ixz = "0" iyy="${m*(3*r*r+h*h)/12}" iyz = "0" izz="${m*r*r/2}" />
+    </xacro:macro>
+    <xacro:macro name="box_inertia" params="m x y z">
+        <inertia ixx="${m*(y*y+z*z)/12}" ixy = "0" ixz = "0" iyy="${m*(x*x+z*z)/12}" iyz = "0" izz="${m*(x*x+z*z)/12}" />
+    </xacro:macro>
+    <xacro:macro name="sphere_inertia" params="m r">
+        <inertia ixx="${2*m*r*r/5}" ixy = "0" ixz = "0" iyy="${2*m*r*r/5}" iyz = "0" izz="${2*m*r*r/5}" />
+    </xacro:macro>
 </robot>

Commit message: update bldc motor

File: materials.xacro (robot description, xacro)
@@ -1,4 +1,5 @@
 <?xml version="1.0"?>
-<robot xmlns:xacro="http://ros.org/wiki/xacro">
+<robot name="materials" xmlns:xacro="http://ros.org/wiki/xacro">
+    <xacro:property name="PI" value="3.14159"/>
     <material name="black">
         <color rgba="0.0 0.0 0.0 1.0"/>

File: sensors/imu_mpu9250/imu_mpu9250.xacro (robot description, xacro)
@@ -32,5 +32,19 @@
         </link>
         <gazebo reference="${prefix}_frame">
+            <gravity>true</gravity>
+            <plugin filename="libhector_gazebo_ros_imu.so" name="gazebo_ros_imu">
+                <bodyName>${prefix}_frame</bodyName>
+                <updateRate>50</updateRate>
+                <serviceName>imu_service</serviceName>
+                <topicName>imu</topicName>
+                <gaussianNoise>0</gaussianNoise>
+                <xyzOffset>0 0 0</xyzOffset>
+                <rpyOffset>0 0 0</rpyOffset>
+            </plugin>
+        </gazebo>
+        <!-- <gazebo reference="${prefix}_frame">
+            <gravity>true</gravity>
             <plugin name="${prefix}_controller" filename="libgazebo_ros_imu.so">
+                <alwaysOn>true</alwaysOn>
                 <topicName>imu/data</topicName>
                 <serviceName>imu/service</serviceName>
@@ -39,5 +53,5 @@
                 <gaussianNoise>0.005</gaussianNoise>
             </plugin>
-        </gazebo>
+        </gazebo> -->
     </xacro:macro>
 </robot>

File: sensors/ydlidar/ydlidar_g4.xacro (robot description, xacro)
@@ -46,6 +46,6 @@
             <sensor type="ray" name="${prefix}_sensor">
                 <pose>0 0 0 0 0 0</pose>
-                <visualize>false</visualize>
-                <update_rate>10</update_rate>
+                <visualize>true</visualize>
+                <update_rate>40</update_rate>
                 <ray>
                     <scan>

Commit message: update lidar g4

File: materials.xacro (robot description, xacro)
@@ -1,7 +1,11 @@
 <?xml version="1.0"?>
-<robot name="materials" xmlns:xacro="http://ros.org/wiki/xacro">
+<robot name="materials"
+    xmlns:xacro="http://ros.org/wiki/xacro">
     <xacro:property name="PI" value="3.14159"/>
     <material name="black">
         <color rgba="0.0 0.0 0.0 1.0"/>
+    </material>
+    <material name="light_black">
+        <color rgba="0.64706 0.61961 0.58824 1"/>
     </material>
     <material name="blue">

File: sensors/imu_mpu9250/imu_mpu9250.xacro (robot description, xacro)
@@ -4,5 +4,4 @@
     <xacro:macro name="imu_mpu9250" params="prefix parent *origin">
         <joint name="${prefix}_fixed" type="fixed">
-            <!-- <origin xyz="0 0 0" rpy="0 0 0"/> -->
             <insert_block name="origin"/>
             <parent link="${parent}"/>
@@ -25,9 +24,4 @@
             </collision>
             <box_inertia m="0.01" x="0.02" y="0.02" z="0.02"/>
-            <!-- <inertial>
-                <mass value="1e-2" />
-                <origin xyz="0 0 0" rpy="0 0 0"/>
-                <inertia ixx="1e-6" ixy="0" ixz="0" iyy="1e-6" iyz="0" izz="1e-6" />
-            </inertial> -->
         </link>
         <gazebo reference="${prefix}_frame">

File: sensors/ydlidar/ydlidar_g4.xacro (robot description, xacro)
@@ -2,5 +2,5 @@
 <robot name="ydlidar_g4"
     xmlns:xacro="http://ros.org/wiki/xacro">
-    <xacro:macro name="ydlidar_g4" params="prefix parent prefix_topic:='fg' *origin min_angle:=-3.14159 max_angle:=3.14159">
+    <xacro:macro name="ydlidar_g4" params="prefix parent prefix_topic *origin min_angle:=-3.14159 max_angle:=3.14159 min_range:=0.26 max_range:=16.0">
         <joint name="${prefix}_base_fixed" type="fixed">
             <!-- <origin xyz="0 0 0" rpy="0 0 0"/> -->
@@ -11,22 +11,21 @@
         <link name="${prefix}_base_link">
             <visual>
-                <origin xyz="0 0 0" rpy="0 0 0" />
+                <origin xyz="0 0 0" rpy="0 0 0"/>
                 <geometry>
                     <mesh filename="package://anman_sensors/sensors/ydlidar/meshes/ydlidar_g4.dae" />
                 </geometry>
-                <material name="">
-                    <color rgba="0.64706 0.61961 0.58824 1" />
-                </material>
+                <material name="light_black"/>
             </visual>
             <collision>
-                <origin xyz="0 0 0" rpy="0 0 0" />
+                <origin xyz="0 0 0.02" rpy="0 0 0"/>
                 <geometry>
-                    <mesh filename="package://anman_sensors/sensors/ydlidar/meshes/ydlidar_g4.dae" />
+                    <cylinder length="0.05" radius="0.040"/>
+                    <!-- <mesh filename="package://anman_sensors/sensors/ydlidar/meshes/ydlidar_g4.dae" /> -->
                 </geometry>
             </collision>
             <inertial>
-                <origin xyz="-0.00029774 0.0066667 0.00013047" rpy="0 0 0" />
+                <origin xyz="-0.00029774 0.0066667 0.00013047" rpy="0 0 0"/>
                 <mass value="0.15717" />
-                <inertia ixx="6.7885E-05" ixy="-1.3987E-07" ixz="-8.1554E-07" iyy="0.00013173" iyz="-9.0932E-08" izz="7.1972E-05" />
+                <inertia ixx="6.7885E-05" ixy="-1.3987E-07" ixz="-8.1554E-07" iyy="0.00013173" iyz="-9.0932E-08" izz="7.1972E-05"/>
             </inertial>
         </link>
@@ -47,9 +46,9 @@
                 <pose>0 0 0 0 0 0</pose>
                 <visualize>true</visualize>
-                <update_rate>40</update_rate>
+                <update_rate>20</update_rate>
                 <ray>
                     <scan>
                         <horizontal>
-                            <samples>720</samples>
+                            <samples>640</samples>
                             <resolution>1</resolution>
                             <min_angle>${min_angle}</min_angle>
@@ -58,15 +57,15 @@
                     </scan>
                     <range>
-                        <min>0.15</min>
-                        <max>15.0</max>
-                        <resolution>0.01</resolution>
+                        <min>${min_range}</min>
+                        <max>${max_range}</max>
+                        <resolution>0.03</resolution>
                     </range>
                     <noise>
                         <type>gaussian</type>
                         <mean>0.0</mean>
-                        <stddev>0.01</stddev>
+                        <stddev>0.0025</stddev>
                     </noise>
                 </ray>
-                <plugin name="gazebo_ros_head_hokuyo_controller" filename="libgazebo_ros_laser.so">
+                <plugin name="${prefix}_gazebo_plugin" filename="libgazebo_ros_laser.so">
                     <topicName>${prefix_topic}/scan</topicName>
                     <frameName>/${prefix}_frame</frameName>

Commit message: add imu

File: materials.xacro (robot description, xacro)
@@ -2,5 +2,5 @@
 <robot name="materials"
     xmlns:xacro="http://ros.org/wiki/xacro">
-    <xacro:property name="PI" value="3.14159"/>
+    <xacro:property name="PI" value="3.1415926535897931"/>
     <material name="black">
         <color rgba="0.0 0.0 0.0 1.0"/>
@@ -16,5 +16,8 @@
     </material>
     <material name="grey">
-        <color rgba="0.2 0.2 0.2 1.0"/>
+        <color rgba="0.75294 0.75294 0.75294 1"/>
+    </material>
+    <material name="dark_grey">
+        <color rgba="0.4 0.4 0.4 1.0"/>
     </material>
     <material name="orange">

File: sensors/imu_mpu9250/imu_mpu9250.xacro (robot description, xacro)
@@ -2,5 +2,5 @@
 <robot name="imu_mpu9250"
     xmlns:xacro="http://ros.org/wiki/xacro">
-    <xacro:macro name="imu_mpu9250" params="prefix parent *origin prefix_topic">
+    <xacro:macro name="imu_mpu9250" params="prefix ns:='' parent *origin">
         <joint name="${prefix}_fixed" type="fixed">
             <insert_block name="origin"/>
@@ -25,10 +25,11 @@
             <box_inertia m="0.01" x="0.02" y="0.02" z="0.02"/>
         </link>
+        <!--
         <gazebo reference="${prefix}_link">
             <gravity>true</gravity>
             <sensor name="${prefix}_sensor" type="imu">
                 <pose>0 0 0 0 0 0</pose>
-                <update_rate>10</update_rate>
-                <plugin  name="${prefix}_gazebo_plugin" filename="libgazebo_ros_imu_sensor.so">
+                <update_rate>100</update_rate>
+                <plugin name="${prefix}_gazebo_plugin" filename="libgazebo_ros_imu_sensor.so">
                     <topicName>${prefix_topic}/imu</topicName>
                     <bodyName>base_link</bodyName>
@@ -40,5 +41,5 @@
                 </plugin>
             </sensor>
-        </gazebo>
+        </gazebo> -->
     </xacro:macro>
 </robot>
